File: Hardware/ws2811-Breakout.sch (EAGLE design)
At the start: 8 parts, among them U1 LED-TRICOLOR-5050

Commit message: v10 Ready for production
Organized files/folders
Added fiducial marks to design
Created panel array of boards for manufacture
v12 now tagged as v10 (initial production ready design)
Parts:
- added FID1, FID2: FIDUCIALUFIDUCIAL, SparkFun-Aesthetics:FIDUCIALUFIDUCIAL
Other:
- note added: "v10"
Changed lines of the file:
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@@
 <part name="GND4" library="SparkFun" deviceset="GND" device=""/>
 <part name="LOGO1" library="SparkFun-Aesthetics" deviceset="OSHW-LOGO" device="S"/>
+<part name="FID1" library="SparkFun-Aesthetics" deviceset="FIDUCIAL" device="UFIDUCIAL"/>
+<part name="FID2" library="SparkFun-Aesthetics" deviceset="FIDUCIAL" device="UFIDUCIAL"/>
 </parts>
 <sheets>
 <sheet>
 <plain>
+<text x="238.76" y="7.62" size="1.778" layer="94">v10</text>
 </plain>
 <instances>
@@
 <instance part="GND4" gate="1" x="175.26" y="96.52"/>
 <instance part="LOGO1" gate="G$1" x="134.62" y="10.16"/>
+<instance part="FID1" gate="G$1" x="241.3" y="27.94"/>
+<instance part="FID2" gate="G$1" x="246.38" y="27.94"/>
 </instances>
 <busses>
