File: Hardware/ws2812-Breakout.brd (EAGLE design)
At the start: 17.8 x 12.7 mm, 10 parts, among them U1 LED-TRICOLOR-5050

Commit message: Updating repo structure, adding firmware, README and .gitignore
Parts:
- added FRAME1: FRAME-LETTER, SparkFun-Aesthetics:CREATIVE_COMMONS
